File: design.kicad_sch (KiCad schematic)
At the start: 14 parts, among them J1 Conn_01x02, J2 Conn_01x02, J3 Conn_01x03, J4 Conn_01x03, U1 TPS61099YFFT

Commit message: DEL Template stuff
Parts:
- removed C1, C2, C3, C4: C_Small, Capacitor_SMD:C_0805_2012Metric, symbol Device:C_Small
- removed J1, J2: Conn_01x02, Connector_PinHeader_2.54mm:PinHeader_1x02_P2.54mm_Vertical, symbol Connector_Generic:Conn_01x02
- removed J3, J4: Conn_01x03, Connector_PinHeader_2.54mm:PinHeader_1x03_P2.54mm_Vertical, symbol Connector_Generic:Conn_01x03
- removed JP1, JP2: SolderJumper_2_Open, Jumper:SolderJumper-2_P1.3mm_Open_RoundedPad1.0x1.5mm, symbol Jumper:SolderJumper_2_Open
- removed L1: L_Small, Inductor_SMD:L_1008_2520Metric, symbol Device:L_Small
- removed R1, R2: R_Small, Resistor_SMD:R_0805_2012Metric, symbol Device:R_Small
- removed U1: TPS61099YFFT, Converter_DCDC_custom:BGA6N40P3X2_122X88X62N, symbol Converter_DCDC_custom:TPS61099YFFT

Commit message: first layouts
Parts:
- added D1, D2, D3, D4, D5, D6, D7, D8, D9: SK6805_1515, LED_SMD:LED_SK6812_EC15_1.5x1.5mm, symbol LED_custom:SK6805_1515
- added J1: Conn_01x03_Female, Connector_PinHeader_2.54mm:PinHeader_1x03_P2.54mm_Horizontal, symbol Connector:Conn_01x03_Female
- added R1: 500, Resistor_SMD:R_0805_2012Metric, symbol Device:R_Small
Connections:
- new net: D3.3 (DOUT), D4.1 (DIN)
- new net: D4.3 (DOUT), D5.1 (DIN)
- new net: D1.3 (DOUT), D2.1 (DIN)
- new net: D2.3 (DOUT), D3.1 (DIN)
- new net: D7.3 (DOUT), D8.1 (DIN)
- new net: D8.3 (DOUT), D9.1 (DIN)
- new net: J1.2 (Pin_2), R1.1
- new net: D5.3 (DOUT), D6.1 (DIN)
- new net: D6.3 (DOUT), D7.1 (DIN)
- new net: D1.1 (DIN), R1.2
- new net GND: D1.4 (VSS), D2.4 (VSS), D3.4 (VSS), D4.4 (VSS), D5.4 (VSS), D6.4 (VSS), D7.4 (VSS), D8.4 (VSS), D9.4 (VSS), J1.1 (Pin_1)
- new net VCC: D1.2 (VDD), D2.2 (VDD), D3.2 (VDD), D4.2 (VDD), D5.2 (VDD), D6.2 (VDD), D7.2 (VDD), D8.2 (VDD), D9.2 (VDD), J1.3 (Pin_3)
